Commit message: demo_resources setup for the cell

File: demo_resources/urdf/ur5e_robot_egp50.urdf.xacro (robot description, xacro)
@@ -10,5 +10,7 @@
   <!-- Instantiate arm + gripper -->
   <xacro:arg name="kinematics_config" default="$(find ur_e_description)/config/ur5e_default.yaml"/>
-  <xacro:ur5e_robot prefix="" joint_limited="false"/>
+  <xacro:ur5e_robot prefix="" joint_limited="false"
+    kinematics_file="${load_yaml('$(arg kinematics_config)')}"
+    />
   <xacro:schunk_egp50 />
   <xacro:cell_ur5e />
@@ -17,5 +19,5 @@
     <parent link="world" />
     <child link = "base_link" />
-    <origin xyz="0.28 0.46 0.01" rpy="0.0 0.0 0.0" />
+    <origin xyz="0.28 0.46 0.01" rpy="0.0 0.0 -1.57" />
   </joint>
   <joint name="world_cell_joint" type="fixed">
